Commit message: Added in velocity and effort control options Added in example setup of control with tide

File: examples/assets/simulation/robot.urdf (robot description, URDF)
Before this commit: robot test_robot, 3 links, 2 joints
Links:
- removed link base_link
- removed link link1
- removed link link2
- added link laser_cut_top_plate, mass 0.631979; collision mesh filename=package://assets/2106_4008_0430.stl; collision mesh filename=package://assets/2106_4008_0430.stl
- added link mock_module, mass 0.0907185; collision mesh filename=package://assets/mock_module.stl; visual mesh filename=package://assets/mock_module.stl
- added link mock_module_2, mass 0.0907185; collision mesh filename=package://assets/mock_module.stl; visual mesh filename=package://assets/mock_module.stl
- added link mock_module_3, mass 0.0907185; collision mesh filename=package://assets/mock_module.stl; visual mesh filename=package://assets/mock_module.stl
- added link mock_module_4, mass 0.0907185; collision mesh filename=package://assets/mock_module.stl; visual mesh filename=package://assets/mock_module.stl
- added link wheel, mass 0.0907185; collision mesh filename=package://assets/wheel.stl; visual mesh filename=package://assets/wheel.stl
- added link wheel_2, mass 0.0907185; collision mesh filename=package://assets/wheel.stl; visual mesh filename=package://assets/wheel.stl
- added link wheel_3, mass 0.0907185; collision mesh filename=package://assets/wheel.stl; visual mesh filename=package://assets/wheel.stl
- added link wheel_4, mass 0.0907185; collision mesh filename=package://assets/wheel.stl; visual mesh filename=package://assets/wheel.stl
Joints:
- removed joint joint1
- removed joint joint2
- added joint fl_drive_wheel: type continuous, parent mock_module_3, child wheel_3, origin xyz=0 0 0 rpy=-1.5708 -0 1.5708, axis 0 0 1, limit effort=10 velocity=10
- added joint fl_steering: type revolute, parent laser_cut_top_plate, child mock_module_3, origin xyz=-0.095885 0.095885 -0.0215 rpy=0 -0 0, axis 0 0 1, limit effort=10 velocity=10
- added joint fr_drive_wheel: type continuous, parent mock_module_4, child wheel_4, origin xyz=0 0 0 rpy=-1.5708 -0 1.5708, axis 0 0 1, limit effort=10 velocity=10
- added joint fr_steering: type revolute, parent laser_cut_top_plate, child mock_module_4, origin xyz=0.095885 0.095885 -0.0215 rpy=0 -0 0, axis 0 0 1, limit effort=10 velocity=10
- added joint rl_drive_wheel: type continuous, parent mock_module, child wheel, origin xyz=0 0 -0.0215 rpy=-1.5708 -0 1.5708, axis 0 0 1, limit effort=10 velocity=10
- added joint rl_steering: type revolute, parent laser_cut_top_plate, child mock_module, origin xyz=-0.095885 -0.095885 0 rpy=0 -0 0, axis 0 0 1, limit effort=10 velocity=10
- added joint rr_drive_wheel: type continuous, parent mock_module_2, child wheel_2, origin xyz=-2.77556e-17 0 0 rpy=-1.5708 -0 1.5708, axis 0 0 1, limit effort=10 velocity=10
- added joint rr_steering: type revolute, parent laser_cut_top_plate, child mock_module_2, origin xyz=0.095885 -0.095885 -0.0215 rpy=0 -0 0, axis 0 0 1, limit effort=10 velocity=10
